Commit message: Remove tooltip collision

File: tm_description/urdf/tm700.urdf.xacro (robot description, xacro)
@@ -260,10 +260,10 @@
     </joint>
     <link name="${prefix}tip_link">
-      <collision>
-        <geometry>
-          <box size="0.05 0.05 0.05"/>
+      <!-- <collision>
+        <geometry>
+          <box size="0 0. 0.025"/>
         </geometry>
         <origin xyz="0 0 0.025" rpy="0 0 0"/>
-      </collision>
+      </collision> -->
     </link>
     <joint name="${prefix}tip_fixed_joint" type="fixed">

Commit message: fix collisions

File: tm_description/urdf/tm700.urdf.xacro (robot description, xacro)
@@ -232,5 +232,5 @@
 	  <mesh filename="package://tm_description/meshes/tm700/visual/Wrist3.STL" />
         </geometry>
-	<origin xyz="0 0 0.015" rpy="0 0 0"/>
+	<origin xyz="0 0 0.012" rpy="0 0 0"/>
         <material name="Grey">
           <color rgba="0.5 0.5 0.5 1.0"/>
@@ -239,6 +239,7 @@
       <collision>
         <geometry>
-	  <mesh filename="package://tm_description/meshes/tm700/collision/wrist_3.STL" />
-        </geometry>
+	  <mesh filename="package://tm_description/meshes/tm700/visual/Wrist3.STL" />
+        </geometry>
+        	<origin xyz="0 0 0.012" rpy="0 0 0"/>
       </collision>
       <xacro:cylinder_inertial radius="0.6" length="0.12" mass="${wrist_3_mass}">
